File: arm_tiny_pcb.kicad_sch (KiCad schematic)
At the start: 26 parts, among them J1 Conn_01x09_Pin, J2 Conn_01x09_Pin, J3 Conn_02x02_Top_Bottom, SW1 SKRKAEE020, SW2 SKRKAEE020, U1 STM32F042F6P6, U2 XBL1117-3.3/STR, U3 USBLC6-2SC6

Commit message: Hardware Rev 2: 20x38.5mm, TVS protection, ME6211 LDO & portable libs
Major hardware revision, project library centralization, and documentation overhaul:

1. Hardware & PCB:
- Updated board dimensions to 20 mm × 38.5 mm (compact, breadboard-friendly layout).
- Added SD05-01FTG TVS diode (SOD-323) on VBUS for ESD and transient surge protection.
- Replaced LDO regulator with low-noise, low-Iq ME6211C33M5G-N (SOT-23-5).
- Replaced tantalum capacitors with MLCC X7R 0805 ceramic capacitors (C1 2.2 µF & C2 1 µF).
- Updated resistor footprints to standard 0402 package (R_0402_1005Metric).
- Optimized power routing, ground stitching vias, and bottom GND return planes.

2. KiCad Libraries & Portability:
- Consolidated project symbols, footprints, and 3D models into self-contained NanoCortex libraries.
- Bundled .wrl 3D models using project-relative paths (${KIPRJMOD}) for seamless multi-machine compatibility.
- Cleaned up obsolete legacy libraries (libs_footprints, libs_symbols).
- Added project library tables (sym-lib-table and fp-lib-table).
- Added .gitignore to exclude KiCad local history, caches, and .lck lock files.

3. Documentation & Media:
- Generated high-quality raytraced 3D renders (top view & isometric perspective).
- Exported vector schematic PDF (arm_tiny_pcb_sch.pdf) and embedded preview graphic.
- Completely overhauled README.md and README_FR.md with full pinout tables, specs, and BOM.
- Expanded roadmap into 3 concrete embedded application tracks: drone telemetry subsystem, hybrid USB-MIDI / op-amp synth, and 40W+ USB-PD Buck converter lab.
Parts:
- removed C1: 10u, Capacitor_Tantalum_SMD:CP_EIA-3528-21_Kemet-B, symbol Device:C_Polarized_Small
- removed C2: 22u, Capacitor_Tantalum_SMD:CP_EIA-3528-21_Kemet-B, symbol Device:C_Polarized_Small
- removed F1: JK-SMD0603-050-6, easyeda2kicad:F0603, symbol easyeda2kicad:JK-SMD0603-050-6
- removed U2: XBL1117-3.3/STR, easyeda2kicad:SOT-89-3_L4.5-W2.4-P1.50-LS4.0-BR, symbol Easyeda2kicad:XBL1117-3.3_STR
- added C1: 2.2u / 25V / X7R, Capacitor_SMD:C_0805_2012Metric, symbol Device:C_Small
- added C2: 1u / 25V / X7R, Capacitor_SMD:C_0805_2012Metric, symbol Device:C_Small
- added D1: SD05-01FTG, NanoCortex:SOD-323_L1.8-W1.3-LS2.5-RD, symbol Device:D_Zener_Small
- added F1: JK-SMD0603-050-6, NanoCortex:F0603, symbol Device:Polyfuse_Small
- added LDO1: ME6211C33M5G-N, NanoCortex:SOT-23-5_L3.0-W1.7-P0.95-LS2.8-BL, symbol NanoCortex:ME6211C33M5G-N
- added R7: 10k, Resistor_SMD:R_0402_1005Metric, symbol Device:R_Small
- LED1: footprint easyeda2kicad:LED0402-R-RD -> NanoCortex:LED0402-R-RD; symbol Easyeda2kicad:16-213_BHC-AN1P2_3T -> NanoCortex:16-213_BHC-AN1P2_3T
- LED2: footprint easyeda2kicad:LED-SMD_4P-L2.0-W2.0-TL_J-ST2020RGB-IC-P4-5-SO1 -> NanoCortex:LED-SMD_4P-L2.0-W2.0-TL_J-ST2020RGB-IC-P4-5-SO1; symbol Easyeda2kicad:SK6805-EC20 -> NanoCortex:SK6805-EC20
- R1, R2, R3, R4, R5, R6: footprint Resistor_SMD:R_01005_0402Metric -> Resistor_SMD:R_0402_1005Metric
- SW1, SW2: footprint easyeda2kicad:SW-SMD_L3.9-W3.0-P4.45 -> NanoCortex:SW-SMD_L3.9-W3.0-P4.45; symbol Easyeda2kicad:SKRKAEE020 -> NanoCortex:SKRKAEE020
- USB1: footprint easyeda2kicad:TYPE-C-SMD_GT-USB-7025 -> NanoCortex:TYPE-C-SMD_GT-USB-7025; symbol easyeda2kicad:GT-USB-7025 -> NanoCortex:GT-USB-7025
Connections:
- net +3.3V: now also C1.1, LDO1.5 (VOUT), R7.1
- net +5V: now also C2.1, F1.2, LDO1.1 (VIN), LDO1.3 (CE)
- net GND: now also C1.2, C2.2, D1.2 (A), LDO1.2 (VSS)
- net NRST: now also R7.2
- net VBUS: now also D1.1 (K), F1.1
- no-connect marks 3 -> 4
Other:
- note added: "Connectors"
- note added: "Linear regulator - 5V -> 3.3V - ME6211C33M5G-N"
- note added: "TVS Diode - SD05-01FTG"
- note removed: "Connector"
- note removed: "Linear regulator - 5V -> 3.3V - XBL1117-3.3/STR"

Commit message: feat(hw): upgrade RGB LED to WS2812B-V6, expose 5V/NRST & introduce CaveRover branding
- Update on-board RGB status LED from SK6805 to WS2812B-2020-V6 for native 3.3V operation
- Add 100 nF decoupling capacitor (C8) adjacent to WS2812B VDD pin
- Update header pinout:
  * Expose protected 5V rail on J1 pin 1 (post-polyfuse F1) for drone receivers and external sensors
  * Expose dedicated hardware NRST on J2 pin 7 for ST-Link "Connect Under Reset" support
  * Complete standard 4-wire SWD debug header (GND, NRST, SWDIO, SWCLK)
- Introduce CaveRover project branding:
  * Add vertical "CAVEROVER" silkscreen text styled in Anurati futuristic font
  * Add custom 8-bit pixel art silkscreen logo footprint (Logo_CaveRover) to NanoCortex.pretty
  * Integrate CaveRover visual identity, badge, and logo into README.md & README_FR.md
- Fix technical inconsistencies in documentation:
  * Remove breadboard-friendly mentions
  * Highlight USART2 (PA2/PA3) as primary user serial port due to PA9/PA10 USB multiplexing
  * Clarify ADC allocation (ADC_IN0 dedicated to RGB LED, 7 external ADC channels available)
  * Add external pull-up warning on PB8 / BOOT0 pin
  * Remove unsupported CAN bus references from drone roadmap in favor of CRSF/SBUS UART
Parts:
- removed LED2: SK6805-EC20, NanoCortex:LED-SMD_4P-L2.0-W2.0-TL_J-ST2020RGB-IC-P4-5-SO1, symbol NanoCortex:SK6805-EC20
- added LED2: WS2812B-2020-V6, NanoCortex:LED-SMD_4P-L2.2-W2.0-P1.00_WS2815C-2020-4P, symbol NanoCortex:WS2812B-2020-V6
Connections:
- net +3.3V: now also LED2.4 (VDD); no longer J1.1 (Pin_1)
- net +5V: now also J1.1 (Pin_1)
- net GND: now also LED2.2 (GND); no longer J2.7 (Pin_7)
- net NRST: now also J2.7 (Pin_7)
- net at R6.2: now also LED2.3 (DI)
Other:
- company: (none) -> Cave Rover
